File: Display_PCB_Rev_1/Display_PCB_Rev_1.brd (EAGLE design)
At the start: 76.5 x 53 mm, 9 parts, among them J1 71430-015

Commit message: VHDCI matched signal length, and Scarab signals wired not matched length
Routing:
- net RXIN0_N: track 73.2 -> 153.2 mm
- net RXIN1_N: track 73.0 -> 147.9 mm
- net RXIN0_P: track 71.8 -> 146.0 mm
- net RXIN1_P: track 71.5 -> 140.6 mm
- net RXIN2_N: track 72.9 -> 137.7 mm
- net RXIN2_P: track 71.3 -> 130.4 mm
- net CLK_N: track 73.0 -> 131.6 mm
- net CLK_P: track 71.3 -> 124.1 mm
Changed lines of the file:
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@@
 <layer number="1" name="Top" color="4" fill="1" visible="yes" active="yes"/>
 <layer number="2" name="Route2" color="1" fill="3" visible="yes" active="yes"/>
-<layer number="3" name="Route3" color="4" fill="3" visible="no" active="yes"/>
+<layer number="3" name="Route3" color="4" fill="3" visible="yes" active="yes"/>
 <layer number="14" name="Route14" color="1" fill="6" visible="no" active="no"/>
 <layer number="15" name="Route15" color="4" fill="6" visible="no" active="no"/>
@@
 <wire x1="49.537615625" y1="54.233003125" x2="34.39735" y2="49.243253125" width="0.127" layer="2"/>
 <wire x1="82.7602375" y1="65.182125" x2="49.537615625" y2="54.233003125" width="0.127" layer="2"/>
-<wire x1="21.9148625" y1="45.12941875" x2="23.06" y2="78.27" width="0" layer="19" extent="1-2"/>
 <wire x1="21.9148625" y1="45.12941875" x2="19.9375" y2="45.125" width="0.127" layer="2"/>
 <wire x1="19.9375" y1="45.125" x2="19.4375" y2="45.8125" width="0.127" layer="2"/>
@@
 <wire x1="18.5625" y1="45.8125" x2="18" y2="45.395" width="0.127" layer="2"/>
 <wire x1="34.39735" y1="49.243253125" x2="21.9148625" y2="45.12941875" width="0.127" layer="2"/>
+<wire x1="23.06" y1="78.27" x2="21.4355" y2="76.7725" width="0.127" layer="3"/>
+<wire x1="21.4355" y1="76.7725" x2="21.4355" y2="73.07239375" width="0.127" layer="3"/>
+<wire x1="21.4355" y1="73.07239375" x2="22.5605" y2="71.94739375" width="0.127" layer="3"/>
+<wire x1="22.5605" y1="71.94739375" x2="22.5605" y2="65.38489375" width="0.127" layer="3"/>
+<wire x1="22.5605" y1="65.38489375" x2="23.38489375" y2="64.5605" width="0.127" layer="3"/>
+<wire x1="23.38489375" y1="64.5605" x2="82.99010625" y2="64.5605" width="0.127" layer="3"/>
+<wire x1="82.99010625" y1="64.5605" x2="83.42960625" y2="65" width="0.127" layer="3"/>
+<wire x1="83.42960625" y1="65" x2="87" y2="65" width="0.127" layer="3"/>
+<wire x1="87" y1="65" x2="87" y2="66" width="0.127" layer="3"/>
 </signal>
 <signal name="RXIN1_N">
@@
 <wire x1="19.3125" y1="50.625" x2="18.8125" y2="50.625" width="0.127" layer="2"/>
 <wire x1="18.8125" y1="50.625" x2="18" y2="50.195" width="0.127" layer="2"/>
-<wire x1="19.3125" y1="50.625" x2="25.6" y2="78.27" width="0" layer="19" extent="1-2"/>
+<wire x1="25.6" y1="78.27" x2="24.3105" y2="77.1075" width="0.127" layer="3"/>
+<wire x1="24.3105" y1="77.1075" x2="24.3105" y2="67.88489375" width="0.127" layer="3"/>
+<wire x1="24.3105" y1="67.88489375" x2="25.13489375" y2="67.0605" width="0.127" layer="3"/>
+<wire x1="25.13489375" y1="67.0605" x2="83.1875" y2="67.0605" width="0.127" layer="3"/>
+<wire x1="83.1875" y1="67.0605" x2="83.1895" y2="67.0625" width="0.127" layer="3"/>
+<wire x1="83.1895" y1="67.0625" x2="87" y2="67.0625" width="0.127" layer="3"/>
+<wire x1="87" y1="67.0625" x2="87" y2="68" width="0.127" layer="3"/>
 </signal>
 <signal name="RXIN0_P">
@@
 <wire x1="38.57133125" y1="51.0274125" x2="21.9375" y2="45.5625" width="0.127" layer="2"/>
 <wire x1="21.9375" y1="45.5625" x2="20.35" y2="45.795" width="0.127" layer="2"/>
-<wire x1="20.35" y1="45.795" x2="23.06" y2="75.73" width="0" layer="19" extent="1-1"/>
+<wire x1="23.06" y1="75.73" x2="21.6895" y2="74.2325" width="0.127" layer="3"/>
+<wire x1="21.6895" y1="74.2325" x2="21.6895" y2="73.17760625" width="0.127" layer="3"/>
+<wire x1="21.6895" y1="73.17760625" x2="22.8145" y2="72.05260625" width="0.127" layer="3"/>
+<wire x1="22.8145" y1="72.05260625" x2="22.8145" y2="65.49010625" width="0.127" layer="3"/>
+<wire x1="22.8145" y1="65.49010625" x2="23.49010625" y2="64.8145" width="0.127" layer="3"/>
+<wire x1="23.49010625" y1="64.8145" x2="82.88489375" y2="64.8145" width="0.127" layer="3"/>
+<wire x1="82.88489375" y1="64.8145" x2="84.07039375" y2="66" width="0.127" layer="3"/>
+<wire x1="84.07039375" y1="66" x2="85" y2="66" width="0.127" layer="3"/>
 </signal>
 <signal name="RXIN1_P">
@@
 <wire x1="43.119925" y1="56.5743875" x2="43.393421875" y2="56.4195" width="0.127" layer="2" curve="90"/>
 <wire x1="43.393421875" y1="56.4195" x2="83.1875" y2="67.4375" width="0.127" layer="2"/>
-<wire x1="21.778046875" y1="50.434734375" x2="25.6" y2="75.73" width="0" layer="19" extent="1-2"/>
+<wire x1="25.6" y1="75.73" x2="24.5645" y2="74.5675" width="0.127" layer="3"/>
+<wire x1="24.5645" y1="74.5675" x2="24.5645" y2="67.99010625" width="0.127" layer="3"/>
+<wire x1="24.5645" y1="67.99010625" x2="25.24010625" y2="67.3145" width="0.127" layer="3"/>
+<wire x1="25.24010625" y1="67.3145" x2="83.1875" y2="67.377" width="0.127" layer="3"/>
+<wire x1="83.1875" y1="67.377" x2="83.873" y2="68" width="0.127" layer="3"/>
+<wire x1="83.873" y1="68" x2="85" y2="68" width="0.127" layer="3"/>
 </signal>
 <signal name="RXIN2_N">
@@
 <wire x1="19.5625" y1="60.0625" x2="18.5" y2="60.4375" width="0.127" layer="2"/>
 <wire x1="18.5" y1="60.4375" x2="16.85" y2="60.595" width="0.127" layer="2"/>
-<wire x1="22.142053125" y1="60.686653125" x2="33.22" y2="78.27" width="0" layer="19" extent="1-2"/>
+<wire x1="33.22" y1="78.27" x2="31.8105" y2="76.9875" width="0.127" layer="3"/>
+<wire x1="31.8105" y1="76.9875" x2="31.8105" y2="71.00989375" width="0.127" layer="3"/>
+<wire x1="31.8105" y1="71.00989375" x2="33.75989375" y2="69.0605" width="0.127" layer="3"/>
+<wire x1="33.75989375" y1="69.0605" x2="82.875" y2="69.0605" width="0.127" layer="3"/>
+<wire x1="82.875" y1="69.0605" x2="82.877" y2="69.0625" width="0.127" layer="3"/>
+<wire x1="82.877" y1="69.0625" x2="86.9375" y2="69.0625" width="0.127" layer="3"/>
+<wire x1="86.9375" y1="69.0625" x2="87" y2="69.125" width="0.127" layer="3"/>
+<wire x1="87" y1="69.125" x2="87" y2="70" width="0.127" layer="3"/>
 </signal>
 <signal name="RXIN2_P">
@@
 <wire x1="53.90419375" y1="65.4012375" x2="82.125" y2="69.3145" width="0.127" layer="2"/>
 <wire x1="19.2" y1="60.995" x2="22.16979375" y2="61.000759375" width="0.127" layer="2"/>
-<wire x1="22.16979375" y1="61.000759375" x2="33.22" y2="75.73" width="0" layer="19" extent="1-2"/>
+<wire x1="33.22" y1="75.73" x2="32.0645" y2="74.4475" width="0.127" layer="3"/>
+<wire x1="32.0645" y1="74.4475" x2="32.0645" y2="71.11510625" width="0.127" layer="3"/>
+<wire x1="32.0645" y1="71.11510625" x2="33.86510625" y2="69.3145" width="0.127" layer="3"/>
+<wire x1="33.86510625" y1="69.3145" x2="82.875" y2="69.3145" width="0.127" layer="3"/>
+<wire x1="82.875" y1="69.3145" x2="83.5605" y2="70" width="0.127" layer="3"/>
+<wire x1="83.5605" y1="70" x2="85" y2="70" width="0.127" layer="3"/>
 </signal>
 <signal name="CLK_N">
@@
 <wire x1="87" y1="74" x2="86.1875" y2="73" width="0.127" layer="2"/>
 <wire x1="86.1875" y1="73" x2="82.578553125" y2="73.06151875" width="0.127" layer="2"/>
-<wire x1="22.300025" y1="65.57076875" x2="35.76" y2="78.27" width="0" layer="19" extent="1-2"/>
+<wire x1="35.76" y1="78.27" x2="34.5605" y2="77.1975" width="0.127" layer="3"/>
+<wire x1="34.5605" y1="77.1975" x2="34.5605" y2="74.00989375" width="0.127" layer="3"/>
+<wire x1="34.5605" y1="74.00989375" x2="35.50989375" y2="73.0605" width="0.127" layer="3"/>
+<wire x1="35.50989375" y1="73.0605" x2="83.25" y2="73.0605" width="0.127" layer="3"/>
+<wire x1="83.25" y1="73.0605" x2="83.252" y2="73.0625" width="0.127" layer="3"/>
+<wire x1="83.252" y1="73.0625" x2="87" y2="73.0625" width="0.127" layer="3"/>
+<wire x1="87" y1="73.0625" x2="87" y2="74" width="0.127" layer="3"/>
 </signal>
 <signal name="CLK_P">
@@
 <wire x1="22.314371875" y1="65.876984375" x2="19.2" y2="65.795" width="0.127" layer="2"/>
 <wire x1="85" y1="74" x2="82.547075" y2="73.376059375" width="0.127" layer="2"/>
-<wire x1="22.314371875" y1="65.876984375" x2="35.76" y2="75.73" width="0" layer="19" extent="1-2"/>
+<wire x1="35.76" y1="75.73" x2="34.8145" y2="74.6575" width="0.127" layer="3"/>
+<wire x1="34.8145" y1="74.6575" x2="34.8145" y2="74.11510625" width="0.127" layer="3"/>
+<wire x1="34.8145" y1="74.11510625" x2="35.61510625" y2="73.3145" width="0.127" layer="3"/>
+<wire x1="35.61510625" y1="73.3145" x2="83.25" y2="73.3145" width="0.127" layer="3"/>
+<wire x1="83.25" y1="73.3145" x2="83.9355" y2="74" width="0.127" layer="3"/>
+<wire x1="83.9355" y1="74" x2="85" y2="74" width="0.127" layer="3"/>
 </signal>
 <signal name="VCC_12">

Commit message: All Differential Pairs with matched lengths
Routing:
- net CLK_P: track 124.1 -> 148.1 mm
- net RXIN2_P: track 130.4 -> 153.2 mm
- net CLK_N: track 131.6 -> 145.9 mm
- net RXIN1_P: track 140.6 -> 152.5 mm
- net RXIN2_N: track 137.7 -> 149.0 mm
- net RXIN0_P: track 146.0 -> 151.0 mm
- net RXIN1_N: track 147.9 -> 152.4 mm
